File: button_pcb/button_pcb.kicad_sch (KiCad schematic)
At the start: 2 parts, among them U1 NRF24L01_Breakout

Commit message: button pcb v0
Parts:
- added 5V_res1, 5V_res2, 5V_res3, 5V_res4, 5V_res5, 5V_res6, GND_button1, GND_res1, GND_res2, GND_res3, GND_res4, GND_res5, GND_res6, J1, J10, J11, J12, J13, J14, J15, J16, J17, J18, J19, J2, J3, J4, J5, J6, J7, J8, J9, V+_arduino1, V-_arduino1, Vin_button1, Vout_button1: Conn_01x01_Pin, Connector_Wire:SolderWire-0.75sqmm_1x01_D1.25mm_OD2.3mm, symbol Connector:Conn_01x01_Pin
- added R_input_button1, R_output5, R_output6, R_output7, R_output8, R_output9: R, Resistor_THT:R_Axial_DIN0207_L6.3mm_D2.5mm_P7.62mm_Horizontal, symbol Device:R
Connections:
- net +5V: now also A1.27 (+5V), 5V_res1.1 (Pin_1), 5V_res2.1 (Pin_1), 5V_res3.1 (Pin_1), 5V_res4.1 (Pin_1), 5V_res5.1 (Pin_1), 5V_res6.1 (Pin_1), Vin_button1.1 (Pin_1); no longer A1.30 (VIN)
- net GND: now also A1.29 (GND), U1.1 (GND), GND_button1.1 (Pin_1), GND_res1.1 (Pin_1), GND_res2.1 (Pin_1), GND_res3.1 (Pin_1), GND_res4.1 (Pin_1), GND_res5.1 (Pin_1), GND_res6.1 (Pin_1); no longer A1.4 (GND)
- net at A1.1 (D1/TX): now also R_output9.2
- net at A1.12 (D9): now also J2.1 (Pin_1)
- net at A1.13 (D10): now also J1.1 (Pin_1)
- net at A1.17 (3V3): now also U1.2 (VCC)
- net at A1.18 (AREF): now also J17.1 (Pin_1)
- net at A1.19 (A0): now also J16.1 (Pin_1)
- net at A1.2 (D0/RX): now also R_output5.2
- net at A1.20 (A1): now also J15.1 (Pin_1)
- net at A1.21 (A2): now also J14.1 (Pin_1)
- net at A1.22 (A3): now also J13.1 (Pin_1)
- net at A1.23 (A4): now also J12.1 (Pin_1)
- net at A1.24 (A5): now also J11.1 (Pin_1)
- net at A1.25 (A6): now also J10.1 (Pin_1)
- net at A1.26 (A7): now also J9.1 (Pin_1)
- net at A1.28 (~{RESET}): now also J19.1 (Pin_1)
- net at A1.3 (~{RESET}): now also J18.1 (Pin_1)
- net at A1.5 (D2): now also R_output8.2
- net at A1.6 (D3): now also R_output7.2
- net at A1.7 (D4): now also R_output6.2
- net at A1.8 (D5): now also J3.1 (Pin_1)
- net at A1.9 (D6): now also R_input_button1.2
- new net: J8.1 (Pin_1), R_output9.1
- new net: A1.30 (VIN), V+_arduino1.1 (Pin_1)
- new net: J6.1 (Pin_1), R_output7.1
- new net: R_input_button1.1, Vout_button1.1 (Pin_1)
- new net: J7.1 (Pin_1), R_output8.1
- new net: J5.1 (Pin_1), R_output6.1
- new net: A1.4 (GND), V-_arduino1.1 (Pin_1)
- new net: J4.1 (Pin_1), R_output5.1
